File: DeVincentiisLinearPSU/DeVincentiisLinearPSU.kicad_sch (KiCad schematic)
At the start: 131 parts, among them J1 0-12-24Vac, J10 V_set, J11 A_set, J2 UPDI, J3 0-24V, J4 Fan 24V, J5 +POW, J6 TP1, J7 +OUT, J8 -POW, J9 I2Csocket, K1 RELAY, Q1 BC817, Q10 BC846, Q11 TIP3055, Q2 BD139, Q3 BC857, Q4 TIP126, Q5 BC846, Q6 TIP3055, Q7 TIP3055, Q8 BC846, Q9 MMBTA06, SW1 EC11, U2 TL081, U3 LM337L_SO8, U4 L7805, U5 TL081, U6 ATtiny3216-S, U7 TL081, U8 MCP4725

Commit message: Value of R49 changed to 330K ohms because with transformers with slightly higher voltage the current limiter had difficulty lowering the output voltage
Parts:
- R49: value 150K -> 330K
Changed lines of the file:
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@@
 	(title_block
 		(title "DeVincentiisDigitalLinearPSU")
-		(date "2025-03-31")
-		(rev "5.0")
+		(date "2025-04-05")
+		(rev "5.1")
 		(company "Antonio de Vincentiis -Pescara - Italy")
 		(comment 1 "Digital Linear Power Supply (DLPS mode)")
@@
 			"AAAAAAAAAAAAAAAAAAAAAAAAAAAAAAAAAAAAAAAAAAAAAAAAAAAAAAAAAAAAAAAAAAAAAAAAAAAA"
 			"AAAAAAAAAAAAAAAAAAAAAAAAAAAAAAAAAAAAAAAAAAAAAAAAAAAAAAAAAAAAAAAAAAAAAAAAAAAA"
+			"AAAAAAAAAAAAAAAAAAAAAAAAAAAAAAAAAAAAAAAAAAAAAAAAAAAAAAAAAAAAAAAAAAAAAAAAAAAA"
+			"AAAAAAAAAAAAAAAAAAAAAAAAAAAAAAAAAAAAAAAAAAAAAAAAAAAAAAAAAAAAAAAAAAAAAAAAAAAA"
+			"AAAAAAAAAAAAAAAAAAAAAAAAAAAAAAAAAAAAAAAAAAAAAAAAAAAAAAAAAAAAAAAAAAAAAAAAAAAA"
+			"AAAAAAAAAAAAAAAAAAAAAAAAAAAAAAAAAAAAAAAAAAAAAAAAAAAAAAAAAAAAAAAAAAAAAAAAAAAA"
+			"AAAAAAAAAAAAAAAAAAAAAAAAAAAAAAAAAAAAAAAAAAAAAAAAAAAAAAAAAAAAAAAAAAAAAAAAAAAA"
+			"AAAAAAAAAAAAAAAAAAAAAAAAAAAAAAAAAAAAAAAAAAAAAAAAAAAAAAAAAAAAAAAAAAAAAAAAAAAA"
+			"AAAAAAAAAAAAAAAAAAAAAAAAAAAAAAAAAAAAAAAAAAAAAAAAAAAAAAAAAAAAAAAAAAAAAAAAAAAA"
+			"AAAAAAAAAAAAAAAAAAAAAAAAAAAAAAAAAAAAAAAAAAAAAAAAAAAAAAAAAAAAAAAAAAAAAAAAAAAA"
+			"AAAAAAAAAAAAAAAAAAAAAAAAAAAAAAAAAAAAAAAAAAAAAAAAAAAAAAAAAAAAAAAAAAAAAAAAAAAA"
+			"AAAAAAAAAAAAAAAAAAAAAAAAAAAAAAAAAAAAAAAAAAAAAAAAAAAAAAAAAAAAAAAAAAAAAAAAAAAA"
+			"AAAAAAAAAAAAAAAAAAAAAAAAAAAAAAAAAAAAAAAAAAAAAAAAAAAAAAAAAAAAAAAAAAAAAAAAAAAA"
+			"AAAAAAAAAAAAAAAAAAAAAAAAAAAAAAAAAAAAAAAAAAAAAAAAAAAAAAAAAAAAAAAAAAAAAAAAAAAA"
+			"AAAAAAAAAAAAAAAAAAAAAAAAAAAAAAAAAAAAAAAAAAAAAAAAAAAAAAAAAAAAAAAAAAAAAAAAAAAA"
+			"AAAAAAAAAAAAAAAAAAAAAAAAAAAAAAAAAAAAAAAAAAAAAAAAAAAAAAAAAAAAAAAAAAAAAAAAAAAA"
+			"AAAAAAAAAAAAAAAAAAAAAAAAAAAAAAAAAAAAAAAAAAAAAAAAAAAAAAAAAAAAAAAAAAAAAAAAAAAA"
+			"AAAAAAAAAAAAAAAAAAAAAAAAAAAAAAAAAAAAAAAAAAAAAAAAAAAAAAAAAAAAAAAAAAAAAAAAAAAA"
+			"AAAAAAAAAAAAAAAAAAAAAAAAAAAAAAAAAAAAAAAAAAAAAAAAAAAAAAAAAAAAAAAAAAAAAAAAAAAA"
+			"AAAAAAAAAAAAAAAAAAAAAAAAAAAAAAAAAAAAAAAAAAAAAAAAAAAAAAAAAAAAAAAAAAAAAAAAAAAA"
 			"AAAAAAAAAAAAAAAAAAAAAAAAAAAAAAAAAAAAAAAAAAAAAA=="
 		)
@@
 			)
 		)
-		(property "Value" "150K"
+		(property "Value" "330K"
 			(at 293.37 92.71 90)
 			(effects

Commit message: I change the mode for self-oscillation prevention by increasing the capacitance of C18 which now works as both integrator/low-pass. Firmware fixed too
Parts:
- removed C19: 100p, Capacitor_SMD:C_1206_3216Metric_Pad1.33x1.80mm_HandSolder, symbol Device:C
- removed C20, C22: 330p, Capacitor_SMD:C_1206_3216Metric_Pad1.33x1.80mm_HandSolder, symbol Device:C
- removed C24: 470p, Capacitor_SMD:C_1206_3216Metric_Pad1.33x1.80mm_HandSolder, symbol Device:C
- removed C28: 0p, Capacitor_SMD:C_1206_3216Metric_Pad1.33x1.80mm_HandSolder, symbol Device:C
- C18: value 470p -> 10n
Other:
- note added: "To scale transformer max voltage increase R1 and R2. EXAMPLES 36V ac : R1=150ohm 3W, R42=82ohm 2W"
- moved on the sheet: R28

Commit message: Fixed PCB errors. Replace C19 and added R51 to prevent self-oscillations
Parts:
- added C19: 1n, Capacitor_SMD:C_1206_3216Metric_Pad1.33x1.80mm_HandSolder, symbol Device:C
- added R51: 1000, Resistor_SMD:R_1206_3216Metric_Pad1.30x1.75mm_HandSolder, symbol Device:R
- R49: value 330K -> 220K
Connections:
- net at Q5.1 (B), Q8.3 (C), R24.2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: now also R23.1; no longer R23.2
- net at R21.1, R28.1, U7.2 (-): now also R51.1
- net at U7.6: now also R23.2, C19.2; no longer R23.1
- new net: C19.1, R51.2
Other:
- moved on the sheet: R23, U7

Commit message: C19 and R51 removed
Parts:
- removed C19: 1n, Capacitor_SMD:C_1206_3216Metric_Pad1.33x1.80mm_HandSolder, symbol Device:C
- removed R51: 1000, Resistor_SMD:R_1206_3216Metric_Pad1.30x1.75mm_HandSolder, symbol Device:R
Changed lines of the file:
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@@
 		(title "DeVincentiisDigitalLinearPSU")
 		(date "2025-04-07")
-		(rev "5.3")
+		(rev "5.4")
 		(company "Antonio de Vincentiis -Pescara - Italy")
 		(comment 1 "Digital Linear Power Supply (DLPS mode)")
@@
 	)
 	(junction
-		(at 269.24 83.82)
-		(diameter 0)
-		(color 0 0 0 0)
-	)
-	(junction
 		(at 337.82 97.79)
 		(diameter 0)
@@
 	)
 	(junction
-		(at 245.11 97.79)
-		(diameter 0)
-		(color 0 0 0 0)
-	)
-	(junction
 		(at 138.43 170.18)
 		(diameter 0)
@@
 	(wire
 		(pts
-			(xy 269.24 92.71) (xy 269.24 97.79)
-		)
-		(stroke
-			(width 0)
-			(type default)
-		)
-	)
-	(wire
-		(pts
 			(xy 314.96 229.87) (xy 321.31 229.87)
 		)
@@
 	(wire
 		(pts
-			(xy 245.11 97.79) (xy 260.35 97.79)
-		)
-		(stroke
-			(width 0)
-			(type default)
-		)
-	)
-	(wire
-		(pts
 			(xy 34.29 201.93) (xy 34.29 214.63)
 		)
@@
 		)
 	)
-	(wire
-		(pts
-			(xy 269.24 83.82) (xy 269.24 85.09)
-		)
-		(stroke
-			(width 0)
-			(type default)
-		)
-	)
 	(polyline
 		(pts
@@
 	(wire
 		(pts
-			(xy 245.11 86.36) (xy 245.11 97.79)
-		)
-		(stroke
-			(width 0)
-			(type default)
-		)
-	)
-	(wire
-		(pts
 			(xy 317.5 224.79) (xy 317.5 242.57)
 		)
@@
 	(wire
 		(pts
-			(xy 245.11 97.79) (xy 245.11 105.41)
+			(xy 245.11 86.36) (xy 245.11 105.41)
 		)
 		(stroke
@@
 		)
 	)
-	(wire
-		(pts
-			(xy 269.24 97.79) (xy 267.97 97.79)
-		)
-		(stroke
-			(width 0)
-			(type default)
-		)
-	)
 	(polyline
 		(pts
@@
 	(wire
 		(pts
-			(xy 262.89 83.82) (xy 269.24 83.82)
+			(xy 262.89 83.82) (xy 278.13 83.82)
 		)
 		(stroke
@@
 	(wire
 		(pts
-			(xy 269.24 83.82) (xy 278.13 83.82)
-		)
-		(stroke
-			(width 0)
-			(type default)
-		)
-	)
-	(wire
-		(pts
 			(xy 309.88 50.8) (xy 317.5 50.8)
 		)
@@
 			"AAAAAAAAAAAAAAAAAAAAAAAAAAAAAAAAAAAAAAAAAAAAAAAAAAAAAAAAAAAAAAAAAAAAAAAAAAAA"
 			"AAAAAAAAAAAAAAAAAAAAAAAAAAAAAAAAAAAAAAAAAAAAAAAAAAAAAAAAAAAAAAAAAAAAAAAAAAAA"
+			"AAAAAAAAAAAAAAAAAAAAAAAAAAAAAAAAAAAAAAAAAAAAAAAAAAAAAAAAAAAAAAAAAAAAAAAAAAAA"
+			"AAAAAAAAAAAAAAAAAAAAAAAAAAAAAAAAAAAAAAAAAAAAAAAAAAAAAAAAAAAAAAAAAAAAAAAAAAAA"
+			"AAAAAAAAAAAAAAAAAAAAAAAAAAAAAAAAAAAAAAAAAAAAAAAAAAAAAAAAAAAAAAAAAAAAAAAAAAAA"
+			"AAAAAAAAAAAAAAAAAAAAAAAAAAAAAAAAAAAAAAAAAAAAAAAAAAAAAAAAAAAAAAAAAAAAAAAAAAAA"
+			"AAAAAAAAAAAAAAAAAAAAAAAAAAAAAAAAAAAAAAAAAAAAAAAAAAAAAAAAAAAAAAAAAAAAAAAAAAAA"
+			"AAAAAAAAAAAAAAAAAAAAAAAAAAAAAAAAAAAAAAAAAAAAAAAAAAAAAAAAAAAAAAAAAAAAAAAAAAAA"
+			"AAAAAAAAAAAAAAAAAAAAAAAAAAAAAAAAAAAAAAAAAAAAAAAAAAAAAAAAAAAAAAAAAAAAAAAAAAAA"
+			"AAAAAAAAAAAAAAAAAAAAAAAAAAAAAAAAAAAAAAAAAAAAAAAAAAAAAAAAAAAAAAAAAAAAAAAAAAAA"
+			"AAAAAAAAAAAAAAAAAAAAAAAAAAAAAAAAAAAAAAAAAAAAAAAAAAAAAAAAAAAAAAAAAAAAAAAAAAAA"
+			"AAAAAAAAAAAAAAAAAAAAAAAAAAAAAAAAAAAAAAAAAAAAAAAAAAAAAAAAAAAAAAAAAAAAAAAAAAAA"
+			"AAAAAAAAAAAAAAAAAAAAAAAAAAAAAAAAAAAAAAAAAAAAAAAAAAAAAAAAAAAAAAAAAAAAAAAAAAAA"
+			"AAAAAAAAAAAAAAAAAAAAAAAAAAAAAAAAAAAAAAAAAAAAAAAAAAAAAAAAAAAAAAAAAAAAAAAAAAAA"
+			"AAAAAAAAAAAAAAAAAAAAAAAAAAAAAAAAAAAAAAAAAAAAAAAAAAAAAAAAAAAAAAAAAAAAAAAAAAAA"
+			"AAAAAAAAAAAAAAAAAAAAAAAAAAAAAAAAAAAAAAAAAAAAAAAAAAAAAAAAAAAAAAAAAAAAAAAAAAAA"
+			"AAAAAAAAAAAAAAAAAAAAAAAAAAAAAAAAAAAAAAAAAAAAAAAAAAAAAAAAAAAAAAAAAAAAAAAAAAAA"
+			"AAAAAAAAAAAAAAAAAAAAAAAAAAAAAAAAAAAAAAAAAAAAAAAAAAAAAAAAAAAAAAAAAAAAAAAAAAAA"
+			"AAAAAAAAAAAAAAAAAAAAAAAAAAAAAAAAAAAAAAAAAAAAAAAAAAAAAAAAAAAAAAAAAAAAAAAAAAAA"
+			"AAAAAAAAAAAAAAAAAAAAAAAAAAAAAAAAAAAAAAAAAAAAAAAAAAAAAAAAAAAAAAAAAAAAAAAAAAAA"
 			"AAAAAAAAAAAAAAAAAAAAAAAAAAAAAAAAAAAAAAAAAAAAAA=="
 		)
@@
 	)
 	(symbol
-		(lib_id "Device:C")
-		(at 269.24 88.9 180)
-		(unit 1)
-		(exclude_from_sim no)
-		(in_bom yes)
-		(on_board yes)
-		(dnp no)
-		(property "Reference" "C19"
-			(at 266.192 86.614 0)
-			(effects
-				(font
-					(size 1.27 1.27)
-				)
-			)
-		)
-		(property "Value" "1n"
-			(at 266.192 91.44 0)
-			(effects
-				(font
-					(size 1.27 1.27)
-				)
-			)
-		)
-		(property "Footprint" "Capacitor_SMD:C_1206_3216Metric_Pad1.33x1.80mm_HandSolder"
-			(at 268.2748 85.09 0)
-			(effects
-				(font
-					(size 1.27 1.27)
-				)
-				(hide yes)
-			)
-		)
-		(property "Datasheet" "~"
-			(at 269.24 88.9 0)
-			(effects
-				(font
-					(size 1.27 1.27)
-				)
-				(hide yes)
-			)
-		)
-		(property "Description" ""
-			(at 269.24 88.9 0)
-			(effects
-				(font
-					(size 1.27 1.27)
-				)
-			)
-		)
-		(pin "1"
-		)
-		(pin "2"
-		)
-		(instances
-			(project "DeVincentiisLinearPSU"
-				(path "/5991d8a9-f3ca-4c4e-8c49-9a8e36fd874b"
-					(reference "C19")
-					(unit 1)
-				)
-			)
-		)
-	)
-	(symbol
 		(lib_id "Device:R")
 		(at 245.11 110.49 0)
@@
 	(symbol
 		(lib_id "Device:R")
-		(at 264.16 97.79 90)
-		(unit 1)
-		(exclude_from_sim no)
-		(in_bom yes)
-		(on_board yes)
-		(dnp no)
-		(property "Reference" "R51"
-			(at 264.414 100.838 90)
-			(effects
-				(font
-					(size 1.27 1.27)
-				)
-			)
-		)
-		(property "Value" "1000"
-			(at 264.16 97.79 90)
-			(effects
-				(font
-					(size 1.27 1.27)
-				)
-			)
-		)
-		(property "Footprint" "Resistor_SMD:R_1206_3216Metric_Pad1.30x1.75mm_HandSolder"
-			(at 264.16 99.568 90)
-			(effects
-				(font
-					(size 1.27 1.27)
-				)
-				(hide yes)
-			)
-		)
-		(property "Datasheet" "~"
-			(at 264.16 97.79 0)
-			(effects
-				(font
-					(size 1.27 1.27)
-				)
-				(hide yes)
-			)
-		)
-		(property "Description" ""
-			(at 264.16 97.79 0)
-			(effects
-				(font
-					(size 1.27 1.27)
-				)
-			)
-		)
-		(pin "1"
-		)
-		(pin "2"
-		)
-		(instances
-			(project "DeVincentiisLinearPSU"
-				(path "/5991d8a9-f3ca-4c4e-8c49-9a8e36fd874b"
-					(reference "R51")
-					(unit 1)
-				)
-			)
-		)
-	)
-	(symbol
-		(lib_id "Device:R")
 		(at 334.01 191.77 180)
 		(unit 1)
@@
 					(size 1.27 1.27)
 				)
+				(hide yes)
 			)
 		)

Commit message: C22 reverted for improve and/or personalize self-oscillations immunity. Added parametric Freecad electronic enclosure
Parts:
- added C22: 330p, Capacitor_SMD:C_1206_3216Metric_Pad1.33x1.80mm_HandSolder, symbol Device:C
Connections:
- net +V out: now also C22.2
- net at R21.1, R28.1, U7.2 (-): now also C22.1
Other:
- company: Antonio de Vincentiis -Pescara - Italy -> Antonio de Vincentiis - Pescara - Italy
- title: DeVincentiisDigitalLinearPSU -> DeVincentiis Digital Linear PS
Changed lines of the file:
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@@
 	(paper "A3")
 	(title_block
-		(title "DeVincentiisDigitalLinearPSU")
-		(date "2025-04-07")
-		(rev "5.4")
-		(company "Antonio de Vincentiis -Pescara - Italy")
+		(title "DeVincentiis Digital Linear PS")
+		(date "2025-04-08")
+		(rev "5.5")
+		(company "Antonio de Vincentiis - Pescara - Italy")
 		(comment 1 "Digital Linear Power Supply (DLPS mode)")
-		(comment 2 "Autoset transformer voltages & single or double winding")
+		(comment 2 "Autoset transformer voltages , single or double winding")
 	)
 	(text "Voltage\noffset"
@@
 	)
 	(junction
+		(at 317.5 105.41)
+		(diameter 0)
+		(color 0 0 0 0)
+	)
+	(junction
 		(at 31.75 149.86)
 		(diameter 0)
@@
 	)
 	(junction
+		(at 331.47 97.79)
+		(diameter 0)
+		(color 0 0 0 0)
+	)
+	(junction
 		(at 119.38 99.06)
 		(diameter 0)
@@
 	(wire
 		(pts
-			(xy 245.11 105.41) (xy 318.77 105.41)
+			(xy 245.11 105.41) (xy 317.5 105.41)
 		)
 		(stroke
@@
 		)
 	)
+	(wire
+		(pts
+			(xy 320.04 97.79) (xy 317.5 97.79)
+		)
+		(stroke
+			(width 0)
+			(type default)
+		)
+	)
 	(polyline
 		(pts
@@
 	(wire
 		(pts
+			(xy 327.66 97.79) (xy 331.47 97.79)
+		)
+		(stroke
+			(width 0)
+			(type default)
+		)
+	)
+	(wire
+		(pts
 			(xy 279.4 228.6) (xy 279.4 217.17)
 		)
@@
 	(wire
 		(pts
+			(xy 317.5 105.41) (xy 318.77 105.41)
+		)
+		(stroke
+			(width 0)
+			(type default)
+		)
+	)
+	(wire
+		(pts
 			(xy 68.58 138.43) (xy 72.39 138.43)
 		)
@@
 	(wire
 		(pts
+			(xy 317.5 97.79) (xy 317.5 105.41)
+		)
+		(stroke
+			(width 0)
+			(type default)
+		)
+	)
+	(wire
+		(pts
 			(xy 82.55 124.46) (xy 82.55 138.43)
 		)
@@
 			"AAAAAAAAAAAAAAAAAAAAAAAAAAAAAAAAAAAAAAAAAAAAAAAAAAAAAAAAAAAAAAAAAAAAAAAAAAAA"
 			"AAAAAAAAAAAAAAAAAAAAAAAAAAAAAAAAAAAAAAAAAAAAAAAAAAAAAAAAAAAAAAAAAAAAAAAAAAAA"
+			"AAAAAAAAAAAAAAAAAAAAAAAAAAAAAAAAAAAAAAAAAAAAAAAAAAAAAAAAAAAAAAAAAAAAAAAAAAAA"
+			"AAAAAAAAAAAAAAAAAAAAAAAAAAAAAAAAAAAAAAAAAAAAAAAAAAAAAAAAAAAAAAAAAAAAAAAAAAAA"
+			"AAAAAAAAAAAAAAAAAAAAAAAAAAAAAAAAAAAAAAAAAAAAAAAAAAAAAAAAAAAAAAAAAAAAAAAAAAAA"
+			"AAAAAAAAAAAAAAAAAAAAAAAAAAAAAAAAAAAAAAAAAAAAAAAAAAAAAAAAAAAAAAAAAAAAAAAAAAAA"
+			"AAAAAAAAAAAAAAAAAAAAAAAAAAAAAAAAAAAAAAAAAAAAAAAAAAAAAAAAAAAAAAAAAAAAAAAAAAAA"
+			"AAAAAAAAAAAAAAAAAAAAAAAAAAAAAAAAAAAAAAAAAAAAAAAAAAAAAAAAAAAAAAAAAAAAAAAAAAAA"
+			"AAAAAAAAAAAAAAAAAAAAAAAAAAAAAAAAAAAAAAAAAAAAAAAAAAAAAAAAAAAAAAAAAAAAAAAAAAAA"
+			"AAAAAAAAAAAAAAAAAAAAAAAAAAAAAAAAAAAAAAAAAAAAAAAAAAAAAAAAAAAAAAAAAAAAAAAAAAAA"
+			"AAAAAAAAAAAAAAAAAAAAAAAAAAAAAAAAAAAAAAAAAAAAAAAAAAAAAAAAAAAAAAAAAAAAAAAAAAAA"
+			"AAAAAAAAAAAAAAAAAAAAAAAAAAAAAAAAAAAAAAAAAAAAAAAAAAAAAAAAAAAAAAAAAAAAAAAAAAAA"
+			"AAAAAAAAAAAAAAAAAAAAAAAAAAAAAAAAAAAAAAAAAAAAAAAAAAAAAAAAAAAAAAAAAAAAAAAAAAAA"
+			"AAAAAAAAAAAAAAAAAAAAAAAAAAAAAAAAAAAAAAAAAAAAAAAAAAAAAAAAAAAAAAAAAAAAAAAAAAAA"
+			"AAAAAAAAAAAAAAAAAAAAAAAAAAAAAAAAAAAAAAAAAAAAAAAAAAAAAAAAAAAAAAAAAAAAAAAAAAAA"
+			"AAAAAAAAAAAAAAAAAAAAAAAAAAAAAAAAAAAAAAAAAAAAAAAAAAAAAAAAAAAAAAAAAAAAAAAAAAAA"
+			"AAAAAAAAAAAAAAAAAAAAAAAAAAAAAAAAAAAAAAAAAAAAAAAAAAAAAAAAAAAAAAAAAAAAAAAAAAAA"
+			"AAAAAAAAAAAAAAAAAAAAAAAAAAAAAAAAAAAAAAAAAAAAAAAAAAAAAAAAAAAAAAAAAAAAAAAAAAAA"
+			"AAAAAAAAAAAAAAAAAAAAAAAAAAAAAAAAAAAAAAAAAAAAAAAAAAAAAAAAAAAAAAAAAAAAAAAAAAAA"
+			"AAAAAAAAAAAAAAAAAAAAAAAAAAAAAAAAAAAAAAAAAAAAAAAAAAAAAAAAAAAAAAAAAAAAAAAAAAAA"
 			"AAAAAAAAAAAAAAAAAAAAAAAAAAAAAAAAAAAAAAAAAAAAAA=="
 		)
@@
 	(symbol
 		(lib_id "Device:C")
+		(at 323.85 97.79 90)
+		(unit 1)
+		(exclude_from_sim no)
+		(in_bom yes)
+		(on_board yes)
+		(dnp no)
+		(property "Reference" "C22"
+			(at 327.152 99.314 90)
+			(effects
+				(font
+					(size 1.27 1.27)
+				)
+			)
+		)
+		(property "Value" "330p"
+			(at 324.358 94.234 90)
+			(effects
+				(font
+					(size 1.27 1.27)
+				)
+			)
+		)
+		(property "Footprint" "Capacitor_SMD:C_1206_3216Metric_Pad1.33x1.80mm_HandSolder"
+			(at 327.66 96.8248 0)
+			(effects
+				(font
+					(size 1.27 1.27)
+				)
+				(hide yes)
+			)
+		)
+		(property "Datasheet" "~"
+			(at 323.85 97.79 0)
+			(effects
+				(font
+					(size 1.27 1.27)
+				)
+				(hide yes)
+			)
+		)
+		(property "Description" ""
+			(at 323.85 97.79 0)
+			(effects
+				(font
+					(size 1.27 1.27)
+				)
+			)
+		)
+		(pin "1"
+		)
+		(pin "2"
+		)
+		(instances
+			(project "DeVincentiisLinearPSU"
+				(path "/5991d8a9-f3ca-4c4e-8c49-9a8e36fd874b"
+					(reference "C22")
+					(unit 1)
+				)
+			)
+		)
+	)
+	(symbol
+		(lib_id "Device:C")
 		(at 165.1 81.28 0)
 		(unit 1)
@@
 		(dnp no)
 		(property "Reference" "R28"
-			(at 322.58 102.87 90)
+			(at 322.072 102.616 90)
 			(effects
 				(font

Commit message: Added R51
Parts:
- added R51: 1000, Resistor_SMD:R_1206_3216Metric_Pad1.30x1.75mm_HandSolder, symbol Device:R
- C22: value 330p -> 10n
Connections:
- net +V out: now also C22.1; no longer C22.2
- net at R21.1, R28.1, U7.2 (-): now also R51.2; no longer C22.1
- new net: C22.2, R51.1
Other:
- moved on the sheet: C22
Changed lines of the file:
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@@
 	(title_block
 		(title "DeVincentiis Digital Linear PS")
-		(date "2025-04-08")
-		(rev "5.5")
+		(date "2025-04-09")
+		(rev "5.6")
 		(company "Antonio de Vincentiis - Pescara - Italy")
 		(comment 1 "Digital Linear Power Supply (DLPS mode)")
@@
 	)
 	(junction
+		(at 337.82 88.9)
+		(diameter 0)
+		(color 0 0 0 0)
+	)
+	(junction
 		(at 43.18 138.43)
 		(diameter 0)
@@
 	)
 	(junction
+		(at 337.82 96.52)
+		(diameter 0)
+		(color 0 0 0 0)
+	)
+	(junction
 		(at 347.98 50.8)
 		(diameter 0)
@@
 	)
 	(junction
-		(at 337.82 97.79)
-		(diameter 0)
-		(color 0 0 0 0)
-	)
-	(junction
 		(at 210.82 138.43)
 		(diameter 0)
@@
 	)
 	(junction
-		(at 331.47 97.79)
-		(diameter 0)
-		(color 0 0 0 0)
-	)
-	(junction
 		(at 119.38 99.06)
 		(diameter 0)
@@
 	(wire
 		(pts
-			(xy 337.82 80.01) (xy 337.82 97.79)
+			(xy 337.82 80.01) (xy 337.82 88.9)
 		)
 		(stroke
@@
 	(wire
 		(pts
+			(xy 318.77 88.9) (xy 317.5 88.9)
+		)
+		(stroke
+			(width 0)
+			(type default)
+		)
+	)
+	(wire
+		(pts
 			(xy 245.11 165.1) (xy 321.31 165.1)
 		)
@@
 	(wire
 		(pts
-			(xy 337.82 100.33) (xy 337.82 97.79)
-		)
-		(stroke
-			(width 0)
-			(type default)
-		)
-	)
-	(wire
-		(pts
 			(xy 31.75 138.43) (xy 31.75 139.7)
 		)
@@
 		)
 	)
-	(wire
-		(pts
-			(xy 320.04 97.79) (xy 317.5 97.79)
-		)
-		(stroke
-			(width 0)
-			(type default)
-		)
-	)
 	(polyline
 		(pts
@@
 	(wire
 		(pts
-			(xy 327.66 97.79) (xy 331.47 97.79)
+			(xy 279.4 228.6) (xy 279.4 217.17)
 		)
 		(stroke
@@
 	(wire
 		(pts
-			(xy 279.4 228.6) (xy 279.4 217.17)
+			(xy 265.43 191.77) (xy 292.1 191.77)
 		)
 		(stroke
@@
 	(wire
 		(pts
-			(xy 265.43 191.77) (xy 292.1 191.77)
+			(xy 133.35 176.53) (xy 138.43 176.53)
 		)
 		(stroke
@@
 	(wire
 		(pts
-			(xy 133.35 176.53) (xy 138.43 176.53)
+			(xy 96.52 176.53) (xy 101.6 176.53)
 		)
 		(stroke
@@
 	(wire
 		(pts
-			(xy 96.52 176.53) (xy 101.6 176.53)
+			(xy 337.82 96.52) (xy 337.82 100.33)
 		)
 		(stroke
@@
 	(wire
 		(pts
-			(xy 331.47 105.41) (xy 331.47 97.79)
+			(xy 331.47 105.41) (xy 331.47 96.52)
 		)
 		(stroke
@@
 	(wire
 		(pts
-			(xy 317.5 97.79) (xy 317.5 105.41)
+			(xy 317.5 88.9) (xy 317.5 105.41)
 		)
 		(stroke
@@
 	(wire
 		(pts
+			(xy 326.39 88.9) (xy 328.93 88.9)
+		)
+		(stroke
+			(width 0)
+			(type default)
+		)
+	)
+	(wire
+		(pts
 			(xy 312.42 125.73) (xy 328.93 125.73)
 		)
@@
 	(wire
 		(pts
+			(xy 337.82 88.9) (xy 337.82 96.52)
+		)
+		(stroke
+			(width 0)
+			(type default)
+		)
+	)
+	(wire
+		(pts
 			(xy 204.47 76.2) (xy 204.47 93.98)
 		)
@@
 	(wire
 		(pts
-			(xy 331.47 97.79) (xy 337.82 97.79)
+			(xy 331.47 96.52) (xy 337.82 96.52)
 		)
 		(stroke
@@
 	(wire
 		(pts
+			(xy 336.55 88.9) (xy 337.82 88.9)
+		)
+		(stroke
+			(width 0)
+			(type default)
+		)
+	)
+	(wire
+		(pts
 			(xy 186.69 176.53) (xy 186.69 205.74)
 		)
@@
 			"AAAAAAAAAAAAAAAAAAAAAAAAAAAAAAAAAAAAAAAAAAAAAAAAAAAAAAAAAAAAAAAAAAAAAAAAAAAA"
 			"AAAAAAAAAAAAAAAAAAAAAAAAAAAAAAAAAAAAAAAAAAAAAAAAAAAAAAAAAAAAAAAAAAAAAAAAAAAA"
+			"AAAAAAAAAAAAAAAAAAAAAAAAAAAAAAAAAAAAAAAAAAAAAAAAAAAAAAAAAAAAAAAAAAAAAAAAAAAA"
+			"AAAAAAAAAAAAAAAAAAAAAAAAAAAAAAAAAAAAAAAAAAAAAAAAAAAAAAAAAAAAAAAAAAAAAAAAAAAA"
+			"AAAAAAAAAAAAAAAAAAAAAAAAAAAAAAAAAAAAAAAAAAAAAAAAAAAAAAAAAAAAAAAAAAAAAAAAAAAA"
+			"AAAAAAAAAAAAAAAAAAAAAAAAAAAAAAAAAAAAAAAAAAAAAAAAAAAAAAAAAAAAAAAAAAAAAAAAAAAA"
+			"AAAAAAAAAAAAAAAAAAAAAAAAAAAAAAAAAAAAAAAAAAAAAAAAAAAAAAAAAAAAAAAAAAAAAAAAAAAA"
+			"AAAAAAAAAAAAAAAAAAAAAAAAAAAAAAAAAAAAAAAAAAAAAAAAAAAAAAAAAAAAAAAAAAAAAAAAAAAA"
+			"AAAAAAAAAAAAAAAAAAAAAAAAAAAAAAAAAAAAAAAAAAAAAAAAAAAAAAAAAAAAAAAAAAAAAAAAAAAA"
+			"AAAAAAAAAAAAAAAAAAAAAAAAAAAAAAAAAAAAAAAAAAAAAAAAAAAAAAAAAAAAAAAAAAAAAAAAAAAA"
+			"AAAAAAAAAAAAAAAAAAAAAAAAAAAAAAAAAAAAAAAAAAAAAAAAAAAAAAAAAAAAAAAAAAAAAAAAAAAA"
+			"AAAAAAAAAAAAAAAAAAAAAAAAAAAAAAAAAAAAAAAAAAAAAAAAAAAAAAAAAAAAAAAAAAAAAAAAAAAA"
+			"AAAAAAAAAAAAAAAAAAAAAAAAAAAAAAAAAAAAAAAAAAAAAAAAAAAAAAAAAAAAAAAAAAAAAAAAAAAA"
+			"AAAAAAAAAAAAAAAAAAAAAAAAAAAAAAAAAAAAAAAAAAAAAAAAAAAAAAAAAAAAAAAAAAAAAAAAAAAA"
+			"AAAAAAAAAAAAAAAAAAAAAAAAAAAAAAAAAAAAAAAAAAAAAAAAAAAAAAAAAAAAAAAAAAAAAAAAAAAA"
+			"AAAAAAAAAAAAAAAAAAAAAAAAAAAAAAAAAAAAAAAAAAAAAAAAAAAAAAAAAAAAAAAAAAAAAAAAAAAA"
+			"AAAAAAAAAAAAAAAAAAAAAAAAAAAAAAAAAAAAAAAAAAAAAAAAAAAAAAAAAAAAAAAAAAAAAAAAAAAA"
+			"AAAAAAAAAAAAAAAAAAAAAAAAAAAAAAAAAAAAAAAAAAAAAAAAAAAAAAAAAAAAAAAAAAAAAAAAAAAA"
+			"AAAAAAAAAAAAAAAAAAAAAAAAAAAAAAAAAAAAAAAAAAAAAAAAAAAAAAAAAAAAAAAAAAAAAAAAAAAA"
+			"AAAAAAAAAAAAAAAAAAAAAAAAAAAAAAAAAAAAAAAAAAAAAAAAAAAAAAAAAAAAAAAAAAAAAAAAAAAA"
 			"AAAAAAAAAAAAAAAAAAAAAAAAAAAAAAAAAAAAAAAAAAAAAA=="
 		)
@@
 	(symbol
 		(lib_id "Device:C")
-		(at 323.85 97.79 90)
+		(at 332.74 88.9 270)
 		(unit 1)
 		(exclude_from_sim no)
@@
 		(dnp no)
 		(property "Reference" "C22"
-			(at 327.152 99.314 90)
+			(at 332.74 92.456 90)
 			(effects
 				(font
@@
 			)
 		)
-		(property "Value" "330p"
-			(at 324.358 94.234 90)
+		(property "Value" "10n"
+			(at 332.74 85.852 90)
 			(effects
 				(font
@@
 		)
 		(property "Footprint" "Capacitor_SMD:C_1206_3216Metric_Pad1.33x1.80mm_HandSolder"
-			(at 327.66 96.8248 0)
+			(at 328.93 89.8652 0)
 			(effects
 				(font
@@
 		)
 		(property "Datasheet" "~"
-			(at 323.85 97.79 0)
+			(at 332.74 88.9 0)
 			(effects
 				(font
@@
 		)
 		(property "Description" ""
-			(at 323.85 97.79 0)
+			(at 332.74 88.9 0)
 			(effects
 				(font
@@
 					(unit 1)
 				)
+			)
+		)
+	)
+	(symbol
+		(lib_id "Device:R")
+		(at 322.58 88.9 270)
+		(unit 1)
+		(exclude_from_sim no)
+		(in_bom yes)
+		(on_board yes)
+		(dnp no)
+		(property "Reference" "R51"
+			(at 322.58 91.44 90)
+			(effects
+				(font
+					(size 1.27 1.27)
+				)
+			)
+		)
+		(property "Value" "1000"
+			(at 322.58 88.9 90)
+			(effects
+				(font
+					(size 1.27 1.27)
+				)
+			)
+		)
+		(property "Footprint" "Resistor_SMD:R_1206_3216Metric_Pad1.30x1.75mm_HandSolder"
+			(at 322.58 87.122 90)
+			(effects
+				(font
+					(size 1.27 1.27)
+				)
+				(hide yes)
+			)
+		)
+		(property "Datasheet" "~"
+			(at 322.58 88.9 0)
+			(effects
+				(font
+					(size 1.27 1.27)
+				)
+				(hide yes)
+			)
+		)
+		(property "Description" ""
+			(at 322.58 88.9 0)
+			(effects
+				(font
+					(size 1.27 1.27)
+				)
+			)
+		)
+		(pin "1"
+		)
+		(pin "2"
+		)
+		(instances
+			(project "DeVincentiisLinearPSU"
+				(path "/5991d8a9-f3ca-4c4e-8c49-9a8e36fd874b"
+					(reference "R51")
+					(unit 1)
+				)
