File: DeVincentiisLinearPSU/DeVincentiisLinearPSU.kicad_sch (KiCad schematic)
At the start: 128 parts, among them J1 0-12-24Vac, J10 V_set, J11 A_set, J2 UPDI, J3 0-24V, J4 Fan 24V, J5 +POW, J6 TP1, J7 +OUT, J8 -POW, J9 I2Csocket, K1 RELAY, Q1 BC817, Q10 BC846, Q11 TIP3055, Q2 BD139, Q3 BC857, Q4 TIP126, Q5 BC846, Q6 TIP3055, Q7 TIP3055, Q8 BC846, Q9 MMBTA06, SW1 EC11, U2 TL081, U3 LM337L_SO8, U4 L7805, U5 TL081, U6 ATtiny3216-S, U7 TL081, U8 MCP4725

Commit message: update notes
Other:
- note added: "1) PREVENT SELF-OSCILLATIONS: since in the event of a short circuit there is a strong tendency to self-oscillate it may be necessary to review (downwards) C18 and/or C22 values 2) SCALE TRANSFORMER VOLTAGE: increase R1 and R2. Example: 36V ac : R1=150ohm 3W, R42=82ohm 3W"
- note added: "3) SCALE CURRENT: add 1 power transistor and 2 resistors every 2A. Furthermore, the values of R12 and R23 must be proportionally decreased as well as appropriately modifying the firmware. L1 will also have to withstand the desired current. Examples: 5 final transistor (10A) R23=15k and R24=1500 2 final transistor (3A) R23=22k and R24=2700"
- note removed: "To scale the current add 1 power transistor and 2 resistors every 2A. Furthermore, the values of R12 and R23 must be proportionally decreased as well as appropriately modifying the firmware. L1 will also have to withstand the desired current. EXAMPLES 5 final transistor (10A) R23=15k and R24=1500 2 final transistor (3A) R23=22k and R24=2700"
- note removed: "To scale transformer max voltage increase R1 and R2. EXAMPLES 36V ac : R1=150ohm 3W, R42=82ohm 2W"
Changed lines of the file:
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@@
 	(title_block
 		(title "DeVincentiis Digital Linear PS")
-		(date "2025-04-09")
-		(rev "5.6")
+		(date "2025-05-02")
+		(rev "5.7")
 		(company "Antonio de Vincentiis - Pescara - Italy")
 		(comment 1 "Digital Linear Power Supply (DLPS mode)")
@@
 		)
 	)
-	(text "To scale transformer max voltage increase R1 and R2. \nEXAMPLES\n36V ac : R1=150ohm 3W, R42=82ohm 2W \n"
+	(text "1) PREVENT SELF-OSCILLATIONS:\nsince in the event of a short circuit \nthere is a strong tendency to self-oscillate \nit may be necessary to review (downwards) \nC18 and/or C22 values\n\n2) SCALE TRANSFORMER VOLTAGE:\nincrease R1 and R2. Example:\n36V ac : R1=150ohm 3W, R42=82ohm 3W \n"
 		(exclude_from_sim no)
-		(at 84.836 22.86 0)
+		(at 101.092 47.752 0)
 		(effects
 			(font
@@
 		)
 	)
-	(text "To scale the current add 1 power transistor and 2 resistors every 2A.\nFurthermore, the values of R12 and R23 must be proportionally decreased \nas well as appropriately modifying the firmware. L1 will also have to\nwithstand the desired current. \nEXAMPLES\n5 final transistor (10A) R23=15k and R24=1500\n2 final transistor (3A) R23=22k and R24=2700"
+	(text "3) SCALE CURRENT:\nadd 1 power transistor and 2 resistors every 2A.\nFurthermore, the values of R12 and R23 must be proportionally decreased \nas well as appropriately modifying the firmware. L1 will also have to\nwithstand the desired current. Examples: \n5 final transistor (10A) R23=15k and R24=1500\n2 final transistor (3A) R23=22k and R24=2700"
 		(exclude_from_sim no)
-		(at 205.232 38.608 0)
+		(at 155.448 42.926 0)
 		(effects
 			(font
@@
 			"AAAAAAAAAAAAAAAAAAAAAAAAAAAAAAAAAAAAAAAAAAAAAAAAAAAAAAAAAAAAAAAAAAAAAAAAAAAA"
 			"AAAAAAAAAAAAAAAAAAAAAAAAAAAAAAAAAAAAAAAAAAAAAAAAAAAAAAAAAAAAAAAAAAAAAAAAAAAA"
+			"AAAAAAAAAAAAAAAAAAAAAAAAAAAAAAAAAAAAAAAAAAAAAAAAAAAAAAAAAAAAAAAAAAAAAAAAAAAA"
+			"AAAAAAAAAAAAAAAAAAAAAAAAAAAAAAAAAAAAAAAAAAAAAAAAAAAAAAAAAAAAAAAAAAAAAAAAAAAA"
+			"AAAAAAAAAAAAAAAAAAAAAAAAAAAAAAAAAAAAAAAAAAAAAAAAAAAAAAAAAAAAAAAAAAAAAAAAAAAA"
+			"AAAAAAAAAAAAAAAAAAAAAAAAAAAAAAAAAAAAAAAAAAAAAAAAAAAAAAAAAAAAAAAAAAAAAAAAAAAA"
+			"AAAAAAAAAAAAAAAAAAAAAAAAAAAAAAAAAAAAAAAAAAAAAAAAAAAAAAAAAAAAAAAAAAAAAAAAAAAA"
+			"AAAAAAAAAAAAAAAAAAAAAAAAAAAAAAAAAAAAAAAAAAAAAAAAAAAAAAAAAAAAAAAAAAAAAAAAAAAA"
+			"AAAAAAAAAAAAAAAAAAAAAAAAAAAAAAAAAAAAAAAAAAAAAAAAAAAAAAAAAAAAAAAAAAAAAAAAAAAA"
+			"AAAAAAAAAAAAAAAAAAAAAAAAAAAAAAAAAAAAAAAAAAAAAAAAAAAAAAAAAAAAAAAAAAAAAAAAAAAA"
+			"AAAAAAAAAAAAAAAAAAAAAAAAAAAAAAAAAAAAAAAAAAAAAAAAAAAAAAAAAAAAAAAAAAAAAAAAAAAA"
+			"AAAAAAAAAAAAAAAAAAAAAAAAAAAAAAAAAAAAAAAAAAAAAAAAAAAAAAAAAAAAAAAAAAAAAAAAAAAA"
+			"AAAAAAAAAAAAAAAAAAAAAAAAAAAAAAAAAAAAAAAAAAAAAAAAAAAAAAAAAAAAAAAAAAAAAAAAAAAA"
+			"AAAAAAAAAAAAAAAAAAAAAAAAAAAAAAAAAAAAAAAAAAAAAAAAAAAAAAAAAAAAAAAAAAAAAAAAAAAA"
+			"AAAAAAAAAAAAAAAAAAAAAAAAAAAAAAAAAAAAAAAAAAAAAAAAAAAAAAAAAAAAAAAAAAAAAAAAAAAA"
+			"AAAAAAAAAAAAAAAAAAAAAAAAAAAAAAAAAAAAAAAAAAAAAAAAAAAAAAAAAAAAAAAAAAAAAAAAAAAA"
+			"AAAAAAAAAAAAAAAAAAAAAAAAAAAAAAAAAAAAAAAAAAAAAAAAAAAAAAAAAAAAAAAAAAAAAAAAAAAA"
+			"AAAAAAAAAAAAAAAAAAAAAAAAAAAAAAAAAAAAAAAAAAAAAAAAAAAAAAAAAAAAAAAAAAAAAAAAAAAA"
+			"AAAAAAAAAAAAAAAAAAAAAAAAAAAAAAAAAAAAAAAAAAAAAAAAAAAAAAAAAAAAAAAAAAAAAAAAAAAA"
+			"AAAAAAAAAAAAAAAAAAAAAAAAAAAAAAAAAAAAAAAAAAAAAAAAAAAAAAAAAAAAAAAAAAAAAAAAAAAA"
 			"AAAAAAAAAAAAAAAAAAAAAAAAAAAAAAAAAAAAAAAAAAAAAA=="
 		)
@@
 		(dnp no)
 		(property "Reference" "R23"
-			(at 275.336 95.25 0)
+			(at 274.574 91.186 0)
 			(effects
 				(font
 					(size 1.27 1.27)
 				)
-				(hide yes)
 			)
 		)

Commit message: DigitalLinearPowerSupply: added C19 (snubber)
Parts:
- added C19: 470n, Capacitor_SMD:C_1206_3216Metric_Pad1.33x1.80mm_HandSolder, symbol Device:C
Connections:
- net +V out: now also C19.1
- net at J3.1 (Pin_1), L1.1: now also C19.2
Changed lines of the file:
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@@
 	(title_block
 		(title "DeVincentiis Digital Linear PS")
-		(date "2025-05-02")
-		(rev "5.7")
+		(date "2025-05-29")
+		(rev "5.8")
 		(company "Antonio de Vincentiis - Pescara - Italy")
 		(comment 1 "Digital Linear Power Supply (DLPS mode)")
@@
 	)
 	(junction
+		(at 360.68 74.93)
+		(diameter 0)
+		(color 0 0 0 0)
+	)
+	(junction
 		(at 31.75 149.86)
 		(diameter 0)
@@
 	)
 	(junction
+		(at 360.68 85.09)
+		(diameter 0)
+		(color 0 0 0 0)
+	)
+	(junction
 		(at 327.66 201.93)
 		(diameter 0)
@@
 	(wire
 		(pts
+			(xy 360.68 85.09) (xy 360.68 97.79)
+		)
+		(stroke
+			(width 0)
+			(type default)
+		)
+	)
+	(wire
+		(pts
 			(xy 44.45 219.71) (xy 44.45 242.57)
 		)
@@
 	(wire
 		(pts
+			(xy 360.68 74.93) (xy 360.68 78.74)
+		)
+		(stroke
+			(width 0)
+			(type default)
+		)
+	)
+	(wire
+		(pts
 			(xy 96.52 218.44) (xy 96.52 242.57)
 		)
@@
 	(wire
 		(pts
+			(xy 355.6 76.2) (xy 355.6 74.93)
+		)
+		(stroke
+			(width 0)
+			(type default)
+		)
+	)
+	(wire
+		(pts
 			(xy 284.48 121.92) (xy 284.48 127)
 		)
@@
 	(wire
 		(pts
+			(xy 355.6 74.93) (xy 360.68 74.93)
+		)
+		(stroke
+			(width 0)
+			(type default)
+		)
+	)
+	(wire
+		(pts
 			(xy 233.68 81.28) (xy 233.68 93.98)
 		)
@@
 	(wire
 		(pts
-			(xy 360.68 50.8) (xy 360.68 78.74)
+			(xy 360.68 50.8) (xy 360.68 74.93)
 		)
 		(stroke
@@
 	(wire
 		(pts
+			(xy 355.6 85.09) (xy 360.68 85.09)
+		)
+		(stroke
+			(width 0)
+			(type default)
+		)
+	)
+	(wire
+		(pts
 			(xy 16.51 149.86) (xy 20.32 149.86)
 		)
@@
 	(wire
 		(pts
+			(xy 355.6 83.82) (xy 355.6 85.09)
+		)
+		(stroke
+			(width 0)
+			(type default)
+		)
+	)
+	(wire
+		(pts
 			(xy 128.27 242.57) (xy 138.43 242.57)
 		)
@@
 	(wire
 		(pts
-			(xy 360.68 81.28) (xy 360.68 97.79)
+			(xy 360.68 81.28) (xy 360.68 85.09)
 		)
 		(stroke
@@
 			"AAAAAAAAAAAAAAAAAAAAAAAAAAAAAAAAAAAAAAAAAAAAAAAAAAAAAAAAAAAAAAAAAAAAAAAAAAAA"
 			"AAAAAAAAAAAAAAAAAAAAAAAAAAAAAAAAAAAAAAAAAAAAAAAAAAAAAAAAAAAAAAAAAAAAAAAAAAAA"
+			"AAAAAAAAAAAAAAAAAAAAAAAAAAAAAAAAAAAAAAAAAAAAAAAAAAAAAAAAAAAAAAAAAAAAAAAAAAAA"
+			"AAAAAAAAAAAAAAAAAAAAAAAAAAAAAAAAAAAAAAAAAAAAAAAAAAAAAAAAAAAAAAAAAAAAAAAAAAAA"
+			"AAAAAAAAAAAAAAAAAAAAAAAAAAAAAAAAAAAAAAAAAAAAAAAAAAAAAAAAAAAAAAAAAAAAAAAAAAAA"
+			"AAAAAAAAAAAAAAAAAAAAAAAAAAAAAAAAAAAAAAAAAAAAAAAAAAAAAAAAAAAAAAAAAAAAAAAAAAAA"
+			"AAAAAAAAAAAAAAAAAAAAAAAAAAAAAAAAAAAAAAAAAAAAAAAAAAAAAAAAAAAAAAAAAAAAAAAAAAAA"
+			"AAAAAAAAAAAAAAAAAAAAAAAAAAAAAAAAAAAAAAAAAAAAAAAAAAAAAAAAAAAAAAAAAAAAAAAAAAAA"
+			"AAAAAAAAAAAAAAAAAAAAAAAAAAAAAAAAAAAAAAAAAAAAAAAAAAAAAAAAAAAAAAAAAAAAAAAAAAAA"
+			"AAAAAAAAAAAAAAAAAAAAAAAAAAAAAAAAAAAAAAAAAAAAAAAAAAAAAAAAAAAAAAAAAAAAAAAAAAAA"
+			"AAAAAAAAAAAAAAAAAAAAAAAAAAAAAAAAAAAAAAAAAAAAAAAAAAAAAAAAAAAAAAAAAAAAAAAAAAAA"
+			"AAAAAAAAAAAAAAAAAAAAAAAAAAAAAAAAAAAAAAAAAAAAAAAAAAAAAAAAAAAAAAAAAAAAAAAAAAAA"
+			"AAAAAAAAAAAAAAAAAAAAAAAAAAAAAAAAAAAAAAAAAAAAAAAAAAAAAAAAAAAAAAAAAAAAAAAAAAAA"
+			"AAAAAAAAAAAAAAAAAAAAAAAAAAAAAAAAAAAAAAAAAAAAAAAAAAAAAAAAAAAAAAAAAAAAAAAAAAAA"
+			"AAAAAAAAAAAAAAAAAAAAAAAAAAAAAAAAAAAAAAAAAAAAAAAAAAAAAAAAAAAAAAAAAAAAAAAAAAAA"
+			"AAAAAAAAAAAAAAAAAAAAAAAAAAAAAAAAAAAAAAAAAAAAAAAAAAAAAAAAAAAAAAAAAAAAAAAAAAAA"
+			"AAAAAAAAAAAAAAAAAAAAAAAAAAAAAAAAAAAAAAAAAAAAAAAAAAAAAAAAAAAAAAAAAAAAAAAAAAAA"
+			"AAAAAAAAAAAAAAAAAAAAAAAAAAAAAAAAAAAAAAAAAAAAAAAAAAAAAAAAAAAAAAAAAAAAAAAAAAAA"
+			"AAAAAAAAAAAAAAAAAAAAAAAAAAAAAAAAAAAAAAAAAAAAAAAAAAAAAAAAAAAAAAAAAAAAAAAAAAAA"
+			"AAAAAAAAAAAAAAAAAAAAAAAAAAAAAAAAAAAAAAAAAAAAAAAAAAAAAAAAAAAAAAAAAAAAAAAAAAAA"
 			"AAAAAAAAAAAAAAAAAAAAAAAAAAAAAAAAAAAAAAAAAAAAAA=="
 		)
@@
 					(unit 1)
 				)
+			)
+		)
+	)
+	(symbol
+		(lib_id "Device:C")
+		(at 355.6 80.01 0)
+		(unit 1)
+		(exclude_from_sim no)
+		(in_bom yes)
+		(on_board yes)
+		(dnp no)
+		(property "Reference" "C19"
+			(at 353.06 77.47 0)
+			(effects
+				(font
+					(size 1.27 1.27)
+				)
+			)
+		)
+		(property "Value" "470n"
+			(at 353.06 82.55 0)
+			(effects
+				(font
+					(size 1.27 1.27)
+				)
+			)
+		)
+		(property "Footprint" "Capacitor_SMD:C_1206_3216Metric_Pad1.33x1.80mm_HandSolder"
+			(at 356.5652 83.82 0)
+			(effects
+				(font
+					(size 1.27 1.27)
+				)
+				(hide yes)
+			)
+		)
+		(property "Datasheet" "~"
+			(at 355.6 80.01 0)
+			(effects
+				(font
+					(size 1.27 1.27)
+				)
+				(hide yes)
+			)
+		)
+		(property "Description" ""
+			(at 355.6 80.01 0)
+			(effects
+				(font
+					(size 1.27 1.27)
+				)
+			)
+		)
+		(pin "1"
+		)
+		(pin "2"
+		)
+		(instances
+			(project "DeVincentiisLinearPSU"
+				(path "/5991d8a9-f3ca-4c4e-8c49-9a8e36fd874b"
+					(reference "C19")
+					(unit 1)
+				)
